Commit message: change wheel123 to left right back

File: tr10_description/urdf/tr10.urdf (robot description, URDF)
Before this commit: robot tr10, 5 links, 4 joints
Links:
- removed link wheel_1
- removed link wheel_2
- removed link wheel_3
- added link wheel_back, mass 0.002; collision sphere radius=0.05; visual sphere radius=0.05
- added link wheel_left, mass 0.2; collision cylinder length=0.05 radius=0.05; visual cylinder length=0.05 radius=0.05
- added link wheel_right, mass 0.2; collision cylinder length=0.05 radius=0.05; visual cylinder length=0.05 radius=0.05
Joints:
- removed joint joint_base_wheel1
- removed joint joint_base_wheel2
- removed joint joint_base_wheel3
- added joint joint_base_wheel_back: type continuous, parent base_link, child wheel_back, origin xyz=-0.1 0 0, axis 0 0 1
- added joint joint_base_wheel_left: type continuous, parent base_link, child wheel_left, origin xyz=0.1 0.1 0, axis 0 1 0
- added joint joint_base_wheel_right: type continuous, parent base_link, child wheel_right, origin xyz=0.1 -0.1 0, axis 0 1 0
